File: DDS_VFO/dds.sch (EAGLE design)
At the start: 48 parts

Commit message: Almost done.
Parts:
- added JP2: (no value), pinhead:PINHD-1X3
Connections:
- removed net BATT+: C65.1, C67.+, U$8.P$1, VREG_5V.VI
- net FILTERED: now also JP2.2
- net GND: now also JP2.1, JP2.3
- net VCC: now also C65.1, C67.+, U$8.P$1, VREG_5V.VI
